Commit message: Feat: Add namespace to sjtu_drone

File: urdf/sjtu_drone.urdf (robot description, URDF)
Before this commit: robot sjtu_drone, 1 links, 0 joints
Links:
- removed link base_link
- added link sjtu_drone/base_link, mass 1.477; collision mesh filename=package://sjtu_drone/meshes/quadrotor_4.stl; visual mesh filename=package://sjtu_drone/meshes/quadrotor_4.dae
- added link sjtu_drone/imu_link, mass 0.01
Joints:
- added joint imu_joint: type fixed, parent sjtu_drone/base_link, child sjtu_drone/imu_link, origin xyz=0 0 0 rpy=0 0 0
