Commit message: Feat: Add specified namespace to published topics

File: urdf/sjtu_drone.0.urdf (robot description, URDF)
Before this commit: robot drone, 2 links, 1 joints
Links:
- removed link drone/base_link
- removed link drone/imu_link
- added link drone0/base_link, mass 1.477; visual mesh filename=package://sjtu_drone/meshes/quadrotor_4.dae
- added link drone0/imu_link, mass 0.01
Joints:
- joint imu_joint: child drone/imu_link -> drone0/imu_link; parent drone/base_link -> drone0/base_link

File: urdf/sjtu_drone.1.urdf (robot description, URDF)
Before this commit: robot drone, 2 links, 1 joints
Links:
- removed link drone/base_link
- removed link drone/imu_link
- added link drone1/base_link, mass 1.477; visual mesh filename=package://sjtu_drone/meshes/quadrotor_4.dae
- added link drone1/imu_link, mass 0.01
Joints:
- joint imu_joint: child drone/imu_link -> drone1/imu_link; parent drone/base_link -> drone1/base_link

File: urdf/sjtu_drone.2.urdf (robot description, URDF)
Before this commit: robot drone, 2 links, 1 joints
Links:
- removed link drone/base_link
- removed link drone/imu_link
- added link drone2/base_link, mass 1.477; visual mesh filename=package://sjtu_drone/meshes/quadrotor_4.dae
- added link drone2/imu_link, mass 0.01
Joints:
- joint imu_joint: child drone/imu_link -> drone2/imu_link; parent drone/base_link -> drone2/base_link

File: urdf/sjtu_drone.3.urdf (robot description, URDF)
Before this commit: robot drone, 2 links, 1 joints
Links:
- removed link drone/base_link
- removed link drone/imu_link
- added link drone3/base_link, mass 1.477; visual mesh filename=package://sjtu_drone/meshes/quadrotor_4.dae
- added link drone3/imu_link, mass 0.01
Joints:
- joint imu_joint: child drone/imu_link -> drone3/imu_link; parent drone/base_link -> drone3/base_link
