Commit message: fix: add 3 more camera for front left right

File: urdf/sjtu_drone_cam.urdf (robot description, URDF)
Before this commit: robot drone, 4 links, 3 joints
Links:
- added link drone/front_camera_link, mass 0.3; collision box size=0.036 0.03 0.03; collision cylinder length=0.042 radius=0.015
- added link drone/front_camera_link_optical
- added link drone/left_camera_link, mass 0.3; collision box size=0.036 0.03 0.03; collision cylinder length=0.042 radius=0.015
- added link drone/left_camera_link_optical
- added link drone/right_camera_link, mass 0.3; collision box size=0.036 0.03 0.03; collision cylinder length=0.042 radius=0.015
- added link drone/right_camera_link_optical
Joints:
- added joint drone/base_to_front_camera_joint: type fixed, parent drone/base_link, child drone/front_camera_link, origin xyz=0.08 0 0 rpy=0 0.24033181 0
- added joint drone/base_to_left_camera_joint: type fixed, parent drone/base_link, child drone/left_camera_link, origin xyz=0.04 -0.04 0 rpy=0 0.24033181 -0.48393994
- added joint drone/base_to_right_camera_joint: type fixed, parent drone/base_link, child drone/right_camera_link, origin xyz=0.04 0.04 0 rpy=0 0.24033181 0.48393994
- added joint drone/front_camera_to_front_camera_link_optical_joint: type fixed, parent drone/front_camera_link, child drone/front_camera_link_optical, origin xyz=0 0 0 rpy=-1.57079632679 0 -1.57079632679
- added joint drone/left_camera_to_left_camera_link_optical_joint: type fixed, parent drone/left_camera_link, child drone/left_camera_link_optical, origin xyz=0 0 0 rpy=-1.57079632679 0 -1.57079632679
- added joint drone/right_camera_to_right_camera_link_optical_joint: type fixed, parent drone/right_camera_link, child drone/right_camera_link_optical, origin xyz=0 0 0 rpy=-1.57079632679 0 -1.57079632679

Commit message: Fix: Rename camera name in `sjtu_drone_cam.urdf`

File: urdf/sjtu_drone_cam.urdf (robot description, URDF)
Before this commit: robot drone, 10 links, 9 joints
Links:
- removed link drone/middle_camera_link
- removed link drone/middle_camera_link_optical
- added link drone/downward_camera_link, mass 0.3; collision box size=0.036 0.03 0.03; collision cylinder length=0.042 radius=0.015
- added link drone/downward_camera_link_optical
Joints:
- removed joint drone/base_to_middle_camera_joint
- removed joint drone/middle_camera_to_middle_camera_link_optical_joint
- added joint drone/base_to_downward_camera_joint: type fixed, parent drone/base_link, child drone/downward_camera_link, origin xyz=0 0 0 rpy=0 1.57079632679 0
- added joint drone/downward_camera_to_downward_camera_link_optical_joint: type fixed, parent drone/downward_camera_link, child drone/downward_camera_link_optical, origin xyz=0 0 0 rpy=-1.57079632679 0 -1.57079632679
- joint drone/base_to_front_camera_joint: origin xyz=0.08 0 0 rpy=0 0.24033181 0 -> xyz=0.14227 0 0 rpy=0 0.366519143 0
- joint drone/base_to_left_camera_joint: origin xyz=0.04 -0.04 0 rpy=0 0.24033181 -0.48393994 -> xyz=0.09942 0.10153 0 rpy=0 0.366519143 0.968657735
- joint drone/base_to_right_camera_joint: origin xyz=0.04 0.04 0 rpy=0 0.24033181 0.48393994 -> xyz=0.09942 -0.10153 0 rpy=0 0.366519143 -0.968657735
